File: Pflanzenuberwachung/Sensoren.kicad_sch (KiCad schematic)
At the start: 0 parts

Commit message: LTE und Sensoren
LTE modul und Ausgänge für Sensoren hinzugefügt
Parts:
- added J3, J5: Conn_01x03_Pin, Connector_PinHeader_2.54mm:PinHeader_1x03_P2.54mm_Vertical, symbol Connector:Conn_01x03_Pin
- added J4: Conn_01x04_Pin, Connector_PinHeader_2.54mm:PinHeader_1x04_P2.54mm_Vertical, symbol Connector:Conn_01x04_Pin
Connections:
- new net ADC_TEMP: J5.2 (Pin_2)
- new net DO_LUX: J3.2 (Pin_2)
- new net GND: J3.3 (Pin_3), J4.4 (Pin_4), J5.3 (Pin_3)
- new net I2C1_SCK_BODEN: J4.3 (Pin_3)
- new net I2C1_SDA_BODEN: J4.2 (Pin_2)
- new net Vout 3,8V: J3.1 (Pin_1), J4.1 (Pin_1), J5.1 (Pin_1)
Other:
- note added: "Anschlussreihenfolge nochmal schauen"
- note added: "Helligkeitssensor sitzt extern"
- note added: "Sensor kommt doch Extern"
- note added: "Temperatursensor"
